File: kicad/smartcard_reader.kicad_sch (KiCad schematic)
At the start: 15 parts, among them J601 7312P0225A13LF, U601 SEC1210/PV-UR2

Commit message: Make the website useful for PCB ordering, sourcing, flashing and card workflows
Parts:
- C603, C604: LCSC C49678 -> C28323; MPN CC0805KRX7R9BB104 -> CL21B105KBFNNNE; Manufacturer YAGEO -> Samsung Electro-Mechanics
Changed lines of the file:
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@@
 			)
 		)
-		(property "Datasheet" "https://www.lcsc.com/datasheet/lcsc_datasheet_2304140030_YAGEO-CC0805KRX7R9BB104_C49678.pdf"
+		(property "Datasheet" "https://www.lcsc.com/datasheet/lcsc_datasheet_2304140030_Samsung-Electro-Mechanics-CL21B105KBFNNNE_C28323.pdf"
 			(at 138.43 115.57 0)
 			(hide yes)
@@
 			)
 		)
-		(property "LCSC" "C49678"
+		(property "LCSC" "C28323"
 			(at 142.24 114.2999 0)
 			(hide yes)
@@
 			)
 		)
-(property "MPN" "CC0805KRX7R9BB104" (at 0 0 0) (effects (font (size 1 1)) (hide yes)))
-(property "Manufacturer" "YAGEO" (at 0 0 0) (effects (font (size 1 1)) (hide yes)))
+(property "MPN" "CL21B105KBFNNNE" (at 0 0 0) (effects (font (size 1 1)) (hide yes)))
+(property "Manufacturer" "Samsung Electro-Mechanics" (at 0 0 0) (effects (font (size 1 1)) (hide yes)))
 )
 	(symbol
@@
 			)
 		)
-		(property "Datasheet" "https://www.lcsc.com/datasheet/lcsc_datasheet_2304140030_YAGEO-CC0805KRX7R9BB104_C49678.pdf"
+		(property "Datasheet" "https://www.lcsc.com/datasheet/lcsc_datasheet_2304140030_Samsung-Electro-Mechanics-CL21B105KBFNNNE_C28323.pdf"
 			(at 128.27 138.43 0)
 			(hide yes)
@@
 			)
 		)
-		(property "LCSC" "C49678"
+		(property "LCSC" "C28323"
 			(at 132.08 137.1599 0)
 			(hide yes)
@@
 			)
 		)
-(property "MPN" "CC0805KRX7R9BB104" (at 0 0 0) (effects (font (size 1 1)) (hide yes)))
-(property "Manufacturer" "YAGEO" (at 0 0 0) (effects (font (size 1 1)) (hide yes)))
+(property "MPN" "CL21B105KBFNNNE" (at 0 0 0) (effects (font (size 1 1)) (hide yes)))
+(property "Manufacturer" "Samsung Electro-Mechanics" (at 0 0 0) (effects (font (size 1 1)) (hide yes)))
 )
 	(symbol
