File: variants/lcd-module-2.8/kicad/buttons.kicad_sch (KiCad schematic)
At the start: 8 parts, among them SW501 TS-1101-C-W, SW502 TS-1101-C-W, SW503 TS-1101-C-W, SW504 TS-1101-C-W, SW505 TS-1101-C-W, SW506 TS-1101-C-W, SW507 TS-1101-C-W, SW508 TS-1101-C-W

Commit message: Revise modular carrier for shared-supplier switches and USB-C
Parts:
- SW501, SW502, SW503, SW504, SW505, SW506, SW507, SW508: value TS-1101-C-W -> PTS636SK25SMTRLFS; footprint ShieldSigner:XKB_TS1101_C_W_reflow -> ShieldSigner:CK_PTS636_SK25_G; LCSC C318938 -> C2689642; MPN TS-1101-C-W -> PTS636SK25SMTRLFS
Changed lines of the file:
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@@
 			)
 		)
-		(property "Value" "TS-1101-C-W"
+		(property "Value" "PTS636SK25SMTRLFS"
 			(at 120.65 113.03 0)
 			(show_name no)
@@
 			)
 		)
-		(property "Footprint" "ShieldSigner:XKB_TS1101_C_W_reflow"
+		(property "Footprint" "ShieldSigner:CK_PTS636_SK25_G"
 			(at 120.65 113.03 0)
 			(hide yes)
@@
 			)
 		)
-		(property "Datasheet" "https://www.lcsc.com/datasheet/lcsc_datasheet_2002271735_XKB-Connection-TS-1101-C-W_C318938.pdf"
+		(property "Datasheet" "https://www.littelfuse.com/assetdocs/littelfuse-ck-tactile-pts636-series-datasheet?assetguid=8a16fd39-1f87-4545-ab06-9e057a0fe304"
 			(at 120.65 113.03 0)
 			(hide yes)
@@
 			)
 		)
-		(property "LCSC" "C318938"
+		(property "LCSC" "C2689642"
 			(at 120.65 110.49 0)
 			(hide yes)
@@
 			)
 		)
-(property "MPN" "TS-1101-C-W" (at 0 0 0) (effects (font (size 1 1)) (hide yes)))
+(property "MPN" "PTS636SK25SMTRLFS" (at 0 0 0) (effects (font (size 1 1)) (hide yes)))
 (property "Manufacturer" "XKB Connection" (at 0 0 0) (effects (font (size 1 1)) (hide yes)))
 )
@@
 			)
 		)
-		(property "Value" "TS-1101-C-W"
+		(property "Value" "PTS636SK25SMTRLFS"
 			(at 120.65 69.85 0)
 			(show_name no)
@@
 			)
 		)
-		(property "Footprint" "ShieldSigner:XKB_TS1101_C_W_reflow"
+		(property "Footprint" "ShieldSigner:CK_PTS636_SK25_G"
 			(at 120.65 69.85 0)
 			(hide yes)
@@
 			)
 		)
-		(property "Datasheet" "https://www.lcsc.com/datasheet/lcsc_datasheet_2002271735_XKB-Connection-TS-1101-C-W_C318938.pdf"
+		(property "Datasheet" "https://www.littelfuse.com/assetdocs/littelfuse-ck-tactile-pts636-series-datasheet?assetguid=8a16fd39-1f87-4545-ab06-9e057a0fe304"
 			(at 120.65 69.85 0)
 			(hide yes)
@@
 			)
 		)
-		(property "LCSC" "C318938"
+		(property "LCSC" "C2689642"
 			(at 120.65 67.31 0)
 			(hide yes)
@@
 			)
 		)
-(property "MPN" "TS-1101-C-W" (at 0 0 0) (effects (font (size 1 1)) (hide yes)))
+(property "MPN" "PTS636SK25SMTRLFS" (at 0 0 0) (effects (font (size 1 1)) (hide yes)))
 (property "Manufacturer" "XKB Connection" (at 0 0 0) (effects (font (size 1 1)) (hide yes)))
 )
@@
 			)
 		)
-		(property "Value" "TS-1101-C-W"
+		(property "Value" "PTS636SK25SMTRLFS"
 			(at 88.9 91.44 0)
 			(show_name no)
@@
 			)
 		)
-		(property "Footprint" "ShieldSigner:XKB_TS1101_C_W_reflow"
+		(property "Footprint" "ShieldSigner:CK_PTS636_SK25_G"
 			(at 88.9 91.44 0)
 			(hide yes)
@@
 			)
 		)
-		(property "Datasheet" "https://www.lcsc.com/datasheet/lcsc_datasheet_2002271735_XKB-Connection-TS-1101-C-W_C318938.pdf"
+		(property "Datasheet" "https://www.littelfuse.com/assetdocs/littelfuse-ck-tactile-pts636-series-datasheet?assetguid=8a16fd39-1f87-4545-ab06-9e057a0fe304"
 			(at 88.9 91.44 0)
 			(hide yes)
@@
 			)
 		)
-		(property "LCSC" "C318938"
+		(property "LCSC" "C2689642"
 			(at 88.9 88.9 0)
 			(hide yes)
@@
 			)
 		)
-(property "MPN" "TS-1101-C-W" (at 0 0 0) (effects (font (size 1 1)) (hide yes)))
+(property "MPN" "PTS636SK25SMTRLFS" (at 0 0 0) (effects (font (size 1 1)) (hide yes)))
 (property "Manufacturer" "XKB Connection" (at 0 0 0) (effects (font (size 1 1)) (hide yes)))
 )
@@
 			)
 		)
-		(property "Value" "TS-1101-C-W"
+		(property "Value" "PTS636SK25SMTRLFS"
 			(at 203.2 92.71 0)
 			(show_name no)
@@
 			)
 		)
-		(property "Footprint" "ShieldSigner:XKB_TS1101_C_W_reflow"
+		(property "Footprint" "ShieldSigner:CK_PTS636_SK25_G"
 			(at 203.2 92.71 0)
 			(hide yes)
@@
 			)
 		)
-		(property "Datasheet" "https://www.lcsc.com/datasheet/lcsc_datasheet_2002271735_XKB-Connection-TS-1101-C-W_C318938.pdf"
+		(property "Datasheet" "https://www.littelfuse.com/assetdocs/littelfuse-ck-tactile-pts636-series-datasheet?assetguid=8a16fd39-1f87-4545-ab06-9e057a0fe304"
 			(at 203.2 92.71 0)
 			(hide yes)
@@
 			)
 		)
-		(property "LCSC" "C318938"
+		(property "LCSC" "C2689642"
 			(at 203.2 90.17 0)
 			(hide yes)
@@
 			)
 		)
-(property "MPN" "TS-1101-C-W" (at 0 0 0) (effects (font (size 1 1)) (hide yes)))
+(property "MPN" "PTS636SK25SMTRLFS" (at 0 0 0) (effects (font (size 1 1)) (hide yes)))
 (property "Manufacturer" "XKB Connection" (at 0 0 0) (effects (font (size 1 1)) (hide yes)))
 )
@@
 			)
 		)
-		(property "Value" "TS-1101-C-W"
+		(property "Value" "PTS636SK25SMTRLFS"
 			(at 120.65 91.44 0)
 			(show_name no)
@@
 			)
 		)
-		(property "Footprint" "ShieldSigner:XKB_TS1101_C_W_reflow"
+		(property "Footprint" "ShieldSigner:CK_PTS636_SK25_G"
 			(at 120.65 91.44 0)
 			(hide yes)
@@
 			)
 		)
-		(property "Datasheet" "https://www.lcsc.com/datasheet/lcsc_datasheet_2002271735_XKB-Connection-TS-1101-C-W_C318938.pdf"
+		(property "Datasheet" "https://www.littelfuse.com/assetdocs/littelfuse-ck-tactile-pts636-series-datasheet?assetguid=8a16fd39-1f87-4545-ab06-9e057a0fe304"
 			(at 120.65 91.44 0)
 			(hide yes)
@@
 			)
 		)
-		(property "LCSC" "C318938"
+		(property "LCSC" "C2689642"
 			(at 120.65 88.9 0)
 			(hide yes)
@@
 			)
 		)
-(property "MPN" "TS-1101-C-W" (at 0 0 0) (effects (font (size 1 1)) (hide yes)))
+(property "MPN" "PTS636SK25SMTRLFS" (at 0 0 0) (effects (font (size 1 1)) (hide yes)))
 (property "Manufacturer" "XKB Connection" (at 0 0 0) (effects (font (size 1 1)) (hide yes)))
 )
@@
 			)
 		)
-		(property "Value" "TS-1101-C-W"
+		(property "Value" "PTS636SK25SMTRLFS"
 			(at 203.2 81.28 0)
 			(show_name no)
@@
 			)
 		)
-		(property "Footprint" "ShieldSigner:XKB_TS1101_C_W_reflow"
+		(property "Footprint" "ShieldSigner:CK_PTS636_SK25_G"
 			(at 203.2 81.28 0)
 			(hide yes)
@@
 			)
 		)
-		(property "Datasheet" "https://www.lcsc.com/datasheet/lcsc_datasheet_2002271735_XKB-Connection-TS-1101-C-W_C318938.pdf"
+		(property "Datasheet" "https://www.littelfuse.com/assetdocs/littelfuse-ck-tactile-pts636-series-datasheet?assetguid=8a16fd39-1f87-4545-ab06-9e057a0fe304"
 			(at 203.2 81.28 0)
 			(hide yes)
@@
 			)
 		)
-		(property "LCSC" "C318938"
+		(property "LCSC" "C2689642"
 			(at 203.2 78.74 0)
 			(hide yes)
@@
 			)
 		)
-(property "MPN" "TS-1101-C-W" (at 0 0 0) (effects (font (size 1 1)) (hide yes)))
+(property "MPN" "PTS636SK25SMTRLFS" (at 0 0 0) (effects (font (size 1 1)) (hide yes)))
 (property "Manufacturer" "XKB Connection" (at 0 0 0) (effects (font (size 1 1)) (hide yes)))
 )
@@
 			)
 		)
-		(property "Value" "TS-1101-C-W"
+		(property "Value" "PTS636SK25SMTRLFS"
 			(at 152.4 91.44 0)
 			(show_name no)
@@
 			)
 		)
-		(property "Footprint" "ShieldSigner:XKB_TS1101_C_W_reflow"
+		(property "Footprint" "ShieldSigner:CK_PTS636_SK25_G"
 			(at 152.4 91.44 0)
 			(hide yes)
@@
 			)
 		)
-		(property "Datasheet" "https://www.lcsc.com/datasheet/lcsc_datasheet_2002271735_XKB-Connection-TS-1101-C-W_C318938.pdf"
+		(property "Datasheet" "https://www.littelfuse.com/assetdocs/littelfuse-ck-tactile-pts636-series-datasheet?assetguid=8a16fd39-1f87-4545-ab06-9e057a0fe304"
 			(at 152.4 91.44 0)
 			(hide yes)
@@
 			)
 		)
-		(property "LCSC" "C318938"
+		(property "LCSC" "C2689642"
 			(at 152.4 88.9 0)
 			(hide yes)
@@
 			)
 		)
-(property "MPN" "TS-1101-C-W" (at 0 0 0) (effects (font (size 1 1)) (hide yes)))
+(property "MPN" "PTS636SK25SMTRLFS" (at 0 0 0) (effects (font (size 1 1)) (hide yes)))
 (property "Manufacturer" "XKB Connection" (at 0 0 0) (effects (font (size 1 1)) (hide yes)))
 )
@@
 			)
 		)
-		(property "Value" "TS-1101-C-W"
+		(property "Value" "PTS636SK25SMTRLFS"
 			(at 203.2 104.14 0)
 			(show_name no)
@@
 			)
 		)
-		(property "Footprint" "ShieldSigner:XKB_TS1101_C_W_reflow"
+		(property "Footprint" "ShieldSigner:CK_PTS636_SK25_G"
 			(at 203.2 104.14 0)
 			(hide yes)
@@
 			)
 		)
-		(property "Datasheet" "https://www.lcsc.com/datasheet/lcsc_datasheet_2002271735_XKB-Connection-TS-1101-C-W_C318938.pdf"
+		(property "Datasheet" "https://www.littelfuse.com/assetdocs/littelfuse-ck-tactile-pts636-series-datasheet?assetguid=8a16fd39-1f87-4545-ab06-9e057a0fe304"
 			(at 203.2 104.14 0)
 			(hide yes)
@@
 			)
 		)
-		(property "LCSC" "C318938"
+		(property "LCSC" "C2689642"
 			(at 203.2 101.6 0)
 			(hide yes)
@@
 			)
 		)
-(property "MPN" "TS-1101-C-W" (at 0 0 0) (effects (font (size 1 1)) (hide yes)))
+(property "MPN" "PTS636SK25SMTRLFS" (at 0 0 0) (effects (font (size 1 1)) (hide yes)))
 (property "Manufacturer" "XKB Connection" (at 0 0 0) (effects (font (size 1 1)) (hide yes)))
 )
