File: variants/lcd-module-2.8/kicad/Power.kicad_sch (KiCad schematic)
At the start: 9 parts, among them J301 TYPE-C 6P(073), J302 Conn_01x02_Pin

Commit message: Rebuild modular signer as an eight-pin 2.8-inch pill carrier
Parts:
- J302: now left out of the parts list
Changed lines of the file:
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@@
 		(body_style 1)
 		(exclude_from_sim no)
-		(in_bom yes)
-		(on_board yes)
+		(in_bom no)
+		(on_board no)
 		(in_pos_files yes)
 		(dnp yes)

Commit message: Revise modular carrier for shared-supplier switches and USB-C
Parts:
- J301: value TYPE-C 6P(073) -> USB4125-GF-A; footprint ShieldSigner:SHOUHAN_TYPE_C_6P_073 -> ShieldSigner:GCT_USB4125_GF_A; LCSC C668623 -> C3151650; MPN TYPE-C 6P(073) -> USB4125-GF-A
Changed lines of the file:
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@@
 			)
 		)
-		(property "Value" "TYPE-C 6P(073)"
+		(property "Value" "USB4125-GF-A"
 			(at 139.7 69.85 0)
 			(show_name no)
@@
 			)
 		)
-		(property "Footprint" "ShieldSigner:SHOUHAN_TYPE_C_6P_073"
+		(property "Footprint" "ShieldSigner:GCT_USB4125_GF_A"
 			(at 143.51 82.55 0)
 			(hide yes)
@@
 			)
 		)
-		(property "Datasheet" "https://www.lcsc.com/datasheet/lcsc_datasheet_2006181823_SHOU-HAN-TYPE-C-6P-073_C668623.pdf"
+		(property "Datasheet" "https://www.gct.co/files/drawings/usb4125.pdf"
 			(at 139.7 85.09 0)
 			(hide yes)
@@
 			)
 		)
-		(property "LCSC" "C668623"
+		(property "LCSC" "C3151650"
 			(at 139.7 67.31 0)
 			(hide yes)
@@
 			)
 		)
-(property "MPN" "TYPE-C 6P(073)" (at 0 0 0) (effects (font (size 1 1)) (hide yes)))
+(property "MPN" "USB4125-GF-A" (at 0 0 0) (effects (font (size 1 1)) (hide yes)))
 (property "Manufacturer" "SHOU HAN" (at 0 0 0) (effects (font (size 1 1)) (hide yes)))
 )

Commit message: Add alternate 5V power header and complete USB-C assembly sourcing
Parts:
- J301: value USB4125-GF-A -> USB4125-GF-A-0190; LCSC C3151650 -> C5246813; MPN USB4125-GF-A -> USB4125-GF-A-0190; Manufacturer SHOU HAN -> GCT
- J302: value Conn_01x02_Pin -> 5V_IN; footprint Connector_PinSocket_2.54mm:PinSocket_1x02_P2.54mm_Vertical -> ShieldSigner:PowerHeader_1x02_P2.54mm; now fitted
Changed lines of the file:
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@@
 			)
 		)
-		(property "Value" "USB4125-GF-A"
+		(property "Value" "USB4125-GF-A-0190"
 			(at 139.7 69.85 0)
 			(show_name no)
@@
 			)
 		)
-		(property "LCSC" "C3151650"
+		(property "LCSC" "C5246813"
 			(at 139.7 67.31 0)
 			(hide yes)
@@
 			)
 		)
-(property "MPN" "USB4125-GF-A" (at 0 0 0) (effects (font (size 1 1)) (hide yes)))
-(property "Manufacturer" "SHOU HAN" (at 0 0 0) (effects (font (size 1 1)) (hide yes)))
+(property "MPN" "USB4125-GF-A-0190" (at 0 0 0) (effects (font (size 1 1)) (hide yes)))
+(property "Manufacturer" "GCT" (at 0 0 0) (effects (font (size 1 1)) (hide yes)))
 )
 	(symbol
@@
 		(exclude_from_sim no)
 		(in_bom no)
-		(on_board no)
-		(in_pos_files yes)
-		(dnp yes)
+		(on_board yes)
+		(in_pos_files no)
+		(dnp no)
 		(property "Reference" "J302"
 			(at 192.786 80.772 0)
@@
 			)
 		)
-		(property "Value" "Conn_01x02_Pin"
+		(property "Value" "5V_IN"
 			(at 189.738 83.058 0)
 			(show_name no)
@@
 			)
 		)
-		(property "Footprint" "Connector_PinSocket_2.54mm:PinSocket_1x02_P2.54mm_Vertical"
+		(property "Footprint" "ShieldSigner:PowerHeader_1x02_P2.54mm"
 			(at 187.96 86.36 0)
 			(hide yes)
